File: Hardware/PCB.brd (EAGLE design)
At the start: 46 x 35 mm, 105 parts, among them IC1 BQ25180YBGR, IC2 DRV2605YZFR, IC3 BMA421, IC9 RT6160AWSC, J1 503480-2400, J2 TC2030-IDC, J4 KH-TYPE-C-16P, Q1 20V/4.2A/52mΩ/1.4W, Q3 SI1308EDL-T1-GE3, U1 NRF52840_QF, U3 MAX17048G+T10, X1 32MHz, X2 32.768kHz

Commit message: solved issue
Parts:
- moved TP_BAT_GND 42.2 mm to (18.3, -5.78)
- moved TP_VBAT 3.65 mm to (14.9, -4.34)
- moved ANT1 0.76 mm to (17.8, 9.95), turned to 0.1 degrees
Routing:
- net GND: track 273.0 -> 68.1 mm, vias 24 -> 8
- net EPD_3V3: track 28.9 -> 14.8 mm, vias 3 -> 2
- net EPD_CS: track 42.4 -> 46.7 mm
- net SWDIO: track 47.0 -> 49.6 mm
- net P1.01: track 56.2 -> 54.6 mm
- net N$7: track 8.35 -> 9.70 mm
- net VBAT: track 26.6 -> 25.7 mm
- added copper zone on layer 1, net GND
- removed copper zone on layer 15, net EPD_3V3
Other:
- outline, holes or cut-outs redrawn
